Commit message: added hand cameras

File: models/urdf/franka_fr3/fr3.urdf (robot description, URDF)
Before this commit: robot fr3, 26 links, 25 joints
Links:
- removed link fr3_hand
- removed link fr3_hand_tcp
- removed link fr3_leftfinger
- removed link fr3_rightfinger
- removed link link0
- removed link link0_accelerometer_bottom
- removed link link0_accelerometer_top
- removed link link1
- removed link link1_accelerometer_bottom
- removed link link1_accelerometer_top
- removed link link2
- removed link link2_accelerometer_bottom
- removed link link2_accelerometer_top
- removed link link3
- removed link link3_accelerometer_bottom
- removed link link3_accelerometer_top
- removed link link4
- removed link link4_accelerometer_bottom
- removed link link4_accelerometer_top
- removed link link5
- removed link link5_accelerometer_bottom
- removed link link5_accelerometer_top
- removed link link6
- removed link link7
- removed link link8
- added link fr3_link0, mass 2.3966; collision mesh filename=package://franka_description/meshes/robots/fr3/collision/li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; visual mesh filename=package://franka_description/meshes/robots/fr3/visual/link0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
- added link fr3_link0_accelerometer_bottom
- added link fr3_link0_accelerometer_top
- added link fr3_link1, mass 2.9274653454; collision mesh filename=package://franka_description/meshes/robots/fr3/collision/li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; visual mesh filename=package://franka_description/meshes/robots/fr3/visual/link1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
- added link fr3_link1_accelerometer_bottom
- added link fr3_link1_accelerometer_top
- added link fr3_link2, mass 2.9355370338; collision mesh filename=package://franka_description/meshes/robots/fr3/collision/li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; visual mesh filename=package://franka_description/meshes/robots/fr3/visual/link2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
- added link fr3_link2_accelerometer_bottom
- added link fr3_link2_accelerometer_top
- added link fr3_link3, mass 2.2449013699; collision mesh filename=package://franka_description/meshes/robots/fr3/collision/li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; visual mesh filename=package://franka_description/meshes/robots/fr3/visual/link3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
- added link fr3_link3_accelerometer_bottom
- added link fr3_link3_accelerometer_top
- added link fr3_link4, mass 2.6155955791; collision mesh filename=package://franka_description/meshes/robots/fr3/collision/li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; visual mesh filename=package://franka_description/meshes/robots/fr3/visual/link4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
- added link fr3_link4_accelerometer_bottom
- added link fr3_link4_accelerometer_top
- added link fr3_link5, mass 2.3271207594; collision mesh filename=package://franka_description/meshes/robots/fr3/collision/li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; visual mesh filename=package://franka_description/meshes/robots/fr3/visual/link5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
- added link fr3_link5_accelerometer_bottom
- added link fr3_link5_accelerometer_top
- added link fr3_link6, mass 1.8170376524; collision mesh filename=package://franka_description/meshes/robots/fr3/collision/li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; visual mesh filename=package://franka_description/meshes/robots/fr3/visual/link6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
- added link fr3_link7, mass 0.6271432862; collision mesh filename=package://franka_description/meshes/robots/fr3/collision/li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; visual mesh filename=package://franka_description/meshes/robots/fr3/visual/link7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
- added link fr3_link8
Joints:
- removed joint base_joint
- removed joint fr3_finger_joint1
- removed joint fr3_finger_joint2
- removed joint fr3_hand_joint
- removed joint fr3_hand_tcp_joint
- removed joint joint1
- removed joint joint2
- removed joint joint3
- removed joint joint4
- removed joint joint5
- removed joint joint6
- removed joint joint7
- removed joint joint8
- removed joint link0_accelerometer_bottom_joint
- removed joint link0_accelerometer_top_joint
- removed joint link1_accelerometer_bottom_joint
- removed joint link1_accelerometer_top_joint
- removed joint link2_accelerometer_bottom_joint
- removed joint link2_accelerometer_top_joint
- removed joint link3_accelerometer_bottom_joint
- removed joint link3_accelerometer_top_joint
- removed joint link4_accelerometer_bottom_joint
- removed joint link4_accelerometer_top_joint
- removed joint link5_accelerometer_bottom_joint
- removed joint link5_accelerometer_top_joint
- added joint fr3_base_joint: type fixed, parent base, child fr3_link0, origin xyz=0 0 0 rpy=0 0 0
- added joint fr3_joint1: type revolute, parent fr3_link0, child fr3_link1, origin xyz=0 0 0.333 rpy=0 0 0, axis 0 0 1, limit lower=-2.9007 upper=2.9007 effort=87.0 velocity=2.62
- added joint fr3_joint2: type revolute, parent fr3_link1, child fr3_link2, origin xyz=0 0 0 rpy=-1.570796326794897 0 0, axis 0 0 1, limit lower=-1.8361 upper=1.8361 effort=87.0 velocity=2.62
- added joint fr3_joint3: type revolute, parent fr3_link2, child fr3_link3, origin xyz=0 -0.316 0 rpy=1.570796326794897 0 0, axis 0 0 1, limit lower=-2.9007 upper=2.9007 effort=87.0 velocity=2.62
- added joint fr3_joint4: type revolute, parent fr3_link3, child fr3_link4, origin xyz=0.0825 0 0 rpy=1.570796326794897 0 0, axis 0 0 1, limit lower=-3.077 upper=-0.1169 effort=87.0 velocity=2.62
- added joint fr3_joint5: type revolute, parent fr3_link4, child fr3_link5, origin xyz=-0.0825 0.384 0 rpy=-1.570796326794897 0 0, axis 0 0 1, limit lower=-2.8763 upper=2.8763 effort=12.0 velocity=5.26
- added joint fr3_joint6: type revolute, parent fr3_link5, child fr3_link6, origin xyz=0 0 0 rpy=1.570796326794897 0 0, axis 0 0 1, limit lower=0.4398 upper=4.6216 effort=12.0 velocity=4.18
- added joint fr3_joint7: type revolute, parent fr3_link6, child fr3_link7, origin xyz=0.088 0 0 rpy=1.570796326794897 0 0, axis 0 0 1, limit lower=-3.0508 upper=3.0508 effort=12.0 velocity=5.26
- added joint fr3_joint8: type fixed, parent fr3_link7, child fr3_link8, origin xyz=0 0 0.107 rpy=0 0 0
- added joint fr3_link0_accelerometer_bottom_joint: type fixed, parent fr3_link0, child fr3_link0_accelerometer_bottom, origin xyz=0 0 0.06 rpy=0 0 0
- added joint fr3_link0_accelerometer_top_joint: type fixed, parent fr3_link0, child fr3_link0_accelerometer_top, origin xyz=0 0 0.05 rpy=3.14159 0 0
- added joint fr3_link1_accelerometer_bottom_joint: type fixed, parent fr3_link1, child fr3_link1_accelerometer_bottom, origin xyz=0 -0.09 0.0 rpy=-1.5708 0 0
- added joint fr3_link1_accelerometer_top_joint: type fixed, parent fr3_link1, child fr3_link1_accelerometer_top, origin xyz=0 -0.1 0.0 rpy=1.5708 0 0
- added joint fr3_link2_accelerometer_bottom_joint: type fixed, parent fr3_link2, child fr3_link2_accelerometer_bottom, origin xyz=0 -0.14 0 rpy=1.5708 0 0
- added joint fr3_link2_accelerometer_top_joint: type fixed, parent fr3_link2, child fr3_link2_accelerometer_top, origin xyz=0 -0.13 0 rpy=-1.5708 0 0
- added joint fr3_link3_accelerometer_bottom_joint: type fixed, parent fr3_link3, child fr3_link3_accelerometer_bottom, origin xyz=0.0825 0.04 0 rpy=1.5708 0 0
- added joint fr3_link3_accelerometer_top_joint: type fixed, parent fr3_link3, child fr3_link3_accelerometer_top, origin xyz=0.0825 0.05 0 rpy=-1.5708 0 0
- added joint fr3_link4_accelerometer_bottom_joint: type fixed, parent fr3_link4, child fr3_link4_accelerometer_bottom, origin xyz=-0.0825 0.06 0 rpy=-1.5708 0 0
- added joint fr3_link4_accelerometer_top_joint: type fixed, parent fr3_link4, child fr3_link4_accelerometer_top, origin xyz=-0.0825 0.05 0 rpy=1.5708 0 0
- added joint fr3_link5_accelerometer_bottom_joint: type fixed, parent fr3_link5, child fr3_link5_accelerometer_bottom, origin xyz=0 0.1 0 rpy=1.5708 0 0
- added joint fr3_link5_accelerometer_top_joint: type fixed, parent fr3_link5, child fr3_link5_accelerometer_top, origin xyz=0 0.11 0 rpy=-1.5708 0 0
